File: KiCad-files/LPC-LQFP100-PitchChangeBoard.sch (KiCad schematic (older format))
At the start: 39 parts, among them CON1 MJ-179P, P1 CONN_02X05, P2 CONN_01X06, SW1 SW_PUSH, SW2 SW_PUSH, U2 LPC11U68JBD100, X1 32.768KHZ, X2 12MHz

Commit message: no message
Parts:
- C1, C10, C11, C12, C13, C14, C15, C16, C17, C18, C19, C2, C20, C3, C4, C5, C6, C7, C8, C9: symbol C -> C-RESCUE-LPC-LQFP100-PitchChangeBoard
- FB1, R3: symbol R -> R-RESCUE-LPC-LQFP100-PitchChangeBoard
